File: Matrice_LED.kicad_sch (KiCad schematic)
At the start: 53 parts

Commit message: Save for the review
Parts:
- removed D102, D52: D, symbol Device:D
- C5: renamed from C4; footprint (none) -> Capacitor_SMD:CP_Elec_6.3x7.7
- R1: footprint (none) -> Resistor_SMD:R_0603_1608Metric_Pad0.98x0.95mm_HandSolder
- renumbered D53 to D1, D28 to D22, D27 to D23, D26 to D24, D24 to D26, D23 to D27, D22 to D28, D42 to D36, D41 to D37, D40 to D38, D38 to D40, D37 to D41, D36 to D42, D96 to D8
Connections:
- net LED_5V: now also C5.1, D1.1 (VDD), D10.1 (VDD), D11.1 (VDD), D12.1 (VDD), D13.1 (VDD), D14.1 (VDD), D15.1 (VDD), D16.1 (VDD), D17.1 (VDD), D18.1 (VDD), D19.1 (VDD), D2.1 (VDD), D20.1 (VDD), D21.1 (VDD), D22.1 (VDD), D23.1 (VDD), D24.1 (VDD), D25.1 (VDD), D26.1 (VDD), D27.1 (VDD), D28.1 (VDD), D29.1 (VDD), D3.1 (VDD), D30.1 (VDD), D31.1 (VDD), D32.1 (VDD), D33.1 (VDD), D34.1 (VDD), D35.1 (VDD), D36.1 (VDD), D37.1 (VDD), D38.1 (VDD), D39.1 (VDD), D4.1 (VDD), D40.1 (VDD), D41.1 (VDD), D42.1 (VDD), D43.1 (VDD), D44.1 (VDD), D45.1 (VDD), D46.1 (VDD), D47.1 (VDD), D48.1 (VDD), D49.1 (VDD), D5.1 (VDD), D6.1 (VDD), D7.1 (VDD), D8.1 (VDD), D9.1 (VDD)
- net LED_GND: now also C5.2, D1.3 (VSS), D10.3 (VSS), D11.3 (VSS), D12.3 (VSS), D13.3 (VSS), D14.3 (VSS), D15.3 (VSS), D16.3 (VSS), D17.3 (VSS), D18.3 (VSS), D19.3 (VSS), D2.3 (VSS), D20.3 (VSS), D21.3 (VSS), D22.3 (VSS), D23.3 (VSS), D24.3 (VSS), D25.3 (VSS), D26.3 (VSS), D27.3 (VSS), D28.3 (VSS), D29.3 (VSS), D3.3 (VSS), D30.3 (VSS), D31.3 (VSS), D32.3 (VSS), D33.3 (VSS), D34.3 (VSS), D35.3 (VSS), D36.3 (VSS), D37.3 (VSS), D38.3 (VSS), D39.3 (VSS), D4.3 (VSS), D40.3 (VSS), D41.3 (VSS), D42.3 (VSS), D43.3 (VSS), D44.3 (VSS), D45.3 (VSS), D46.3 (VSS), D47.3 (VSS), D48.3 (VSS), D49.3 (VSS), D5.3 (VSS), D6.3 (VSS), D7.3 (VSS), D8.3 (VSS), D9.3 (VSS)
Changed lines of the file:
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@@
 	(wire
 		(pts
-			(xy 309.88 236.22) (xy 309.88 237.49)
+			(xy 309.88 227.33) (xy 309.88 237.49)
 		)
 		(stroke
@@
 	(wire
 		(pts
-			(xy 76.2 48.26) (xy 76.2 50.8)
+			(xy 76.2 38.1) (xy 76.2 50.8)
 		)
 		(stroke
@@
 	(wire
 		(pts
-			(xy 76.2 38.1) (xy 76.2 40.64)
-		)
-		(stroke
-			(width 0)
-			(type default)
-		)
-	)
-	(wire
-		(pts
 			(xy 194.31 50.8) (xy 194.31 55.88)
 		)
@@
 	(wire
 		(pts
-			(xy 309.88 227.33) (xy 309.88 228.6)
-		)
-		(stroke
-			(width 0)
-			(type default)
-		)
-	)
-	(wire
-		(pts
 			(xy 143.51 101.6) (xy 168.91 101.6)
 		)
@@
 		(dnp no)
 		(fields_autoplaced yes)
-		(property "Reference" "D96"
+		(property "Reference" "D8"
 			(at 281.94 83.4546 0)
 			(effects
@@
 			(project ""
 				(path "/88219bad-2ec7-47f4-a09d-0e9b2dfe4690/b16f55a3-e312-45fa-a45f-1850db188063"
-					(reference "D96")
+					(reference "D8")
 					(unit 1)
 				)
@@
 		(dnp no)
 		(fields_autoplaced yes)
-		(property "Reference" "D41"
+		(property "Reference" "D37"
 			(at 256.54 185.0546 0)
 			(effects
@@
 			(project "Projet-ELEC-GISTRE"
 				(path "/88219bad-2ec7-47f4-a09d-0e9b2dfe4690/b16f55a3-e312-45fa-a45f-1850db188063"
-					(reference "D41")
+					(reference "D37")
 					(unit 1)
 				)
@@
 	)
 	(symbol
-		(lib_id "Device:D")
-		(at 76.2 44.45 90)
-		(unit 1)
-		(exclude_from_sim no)
-		(in_bom yes)
-		(on_board yes)
-		(dnp no)
-		(fields_autoplaced yes)
-		(property "Reference" "D52"
-			(at 78.74 43.1799 90)
-			(effects
-				(font
-					(size 1.27 1.27)
-				)
-				(justify right)
-			)
-		)
-		(property "Value" "D"
-			(at 78.74 45.7199 90)
-			(effects
-				(font
-					(size 1.27 1.27)
-				)
-				(justify right)
-			)
-		)
-		(property "Footprint" ""
-			(at 76.2 44.45 0)
-			(effects
-				(font
-					(size 1.27 1.27)
-				)
-				(hide yes)
-			)
-		)
-		(property "Datasheet" "~"
-			(at 76.2 44.45 0)
-			(effects
-				(font
-					(size 1.27 1.27)
-				)
-				(hide yes)
-			)
-		)
-		(property "Description" "Diode"
-			(at 76.2 44.45 0)
-			(effects
-				(font
-					(size 1.27 1.27)
-				)
-				(hide yes)
-			)
-		)
-		(property "Sim.Device" "D"
-			(at 76.2 44.45 0)
-			(effects
-				(font
-					(size 1.27 1.27)
-				)
-				(hide yes)
-			)
-		)
-		(property "Sim.Pins" "1=K 2=A"
-			(at 76.2 44.45 0)
-			(effects
-				(font
-					(size 1.27 1.27)
-				)
-				(hide yes)
-			)
-		)
-		(pin "1"
-		)
-		(pin "2"
-		)
-		(instances
-			(project ""
-				(path "/88219bad-2ec7-47f4-a09d-0e9b2dfe4690/b16f55a3-e312-45fa-a45f-1850db188063"
-					(reference "D52")
-					(unit 1)
-				)
-			)
-		)
-	)
-	(symbol
 		(lib_id "LED:WS2812B")
 		(at 270.51 114.3 0)
@@
 		(dnp no)
 		(fields_autoplaced yes)
-		(property "Reference" "D23"
+		(property "Reference" "D27"
 			(at 154.94 134.2546 0)
 			(effects
@@
 			(project "Projet-ELEC-GISTRE"
 				(path "/88219bad-2ec7-47f4-a09d-0e9b2dfe4690/b16f55a3-e312-45fa-a45f-1850db188063"
-					(reference "D23")
+					(reference "D27")
 					(unit 1)
 				)
@@
 			)
 		)
-		(property "Footprint" ""
+		(property "Footprint" "Resistor_SMD:R_0603_1608Metric_Pad0.98x0.95mm_HandSolder"
 			(at 104.14 65.278 90)
 			(effects
@@
 		(dnp no)
 		(fields_autoplaced yes)
-		(property "Reference" "D38"
+		(property "Reference" "D40"
 			(at 180.34 185.0546 0)
 			(effects
@@
 			(project "Projet-ELEC-GISTRE"
 				(path "/88219bad-2ec7-47f4-a09d-0e9b2dfe4690/b16f55a3-e312-45fa-a45f-1850db188063"
-					(reference "D38")
+					(reference "D40")
 					(unit 1)
 				)
@@
 		(dnp no)
 		(fields_autoplaced yes)
-		(property "Reference" "C4"
+		(property "Reference" "C5"
 			(at 313.69 56.2609 0)
 			(effects
@@
 			)
 		)
-		(property "Footprint" ""
+		(property "Footprint" "Capacitor_SMD:CP_Elec_6.3x7.7"
 			(at 310.8452 62.23 0)
 			(effects
@@
 			(project ""
 				(path "/88219bad-2ec7-47f4-a09d-0e9b2dfe4690/b16f55a3-e312-45fa-a45f-1850db188063"
-					(reference "C4")
+					(reference "C5")
 					(unit 1)
 				)
@@
 		(dnp no)
 		(fields_autoplaced yes)
-		(property "Reference" "D26"
+		(property "Reference" "D24"
 			(at 231.14 134.2546 0)
 			(effects
@@
 			(project "Projet-ELEC-GISTRE"
 				(path "/88219bad-2ec7-47f4-a09d-0e9b2dfe4690/b16f55a3-e312-45fa-a45f-1850db188063"
-					(reference "D26")
+					(reference "D24")
 					(unit 1)
 				)
@@
 		(dnp no)
 		(fields_autoplaced yes)
-		(property "Reference" "D22"
+		(property "Reference" "D28"
 			(at 129.54 134.2546 0)
 			(effects
@@
 			(project "Projet-ELEC-GISTRE"
 				(path "/88219bad-2ec7-47f4-a09d-0e9b2dfe4690/b16f55a3-e312-45fa-a45f-1850db188063"
-					(reference "D22")
+					(reference "D28")
 					(unit 1)
 				)
@@
 		(dnp no)
 		(fields_autoplaced yes)
-		(property "Reference" "D28"
+		(property "Reference" "D22"
 			(at 281.94 134.2546 0)
 			(effects
@@
 			(project "Projet-ELEC-GISTRE"
 				(path "/88219bad-2ec7-47f4-a09d-0e9b2dfe4690/b16f55a3-e312-45fa-a45f-1850db188063"
-					(reference "D28")
+					(reference "D22")
 					(unit 1)
 				)
@@
 		(dnp no)
 		(fields_autoplaced yes)
-		(property "Reference" "D37"
+		(property "Reference" "D41"
 			(at 154.94 185.0546 0)
 			(effects
@@
 			(project "Projet-ELEC-GISTRE"
 				(path "/88219bad-2ec7-47f4-a09d-0e9b2dfe4690/b16f55a3-e312-45fa-a45f-1850db188063"
-					(reference "D37")
+					(reference "D41")
 					(unit 1)
 				)
@@
 		(dnp no)
 		(fields_autoplaced yes)
-		(property "Reference" "D53"
+		(property "Reference" "D1"
 			(at 129.54 57.0798 0)
 			(effects
@@
 			(project ""
 				(path "/88219bad-2ec7-47f4-a09d-0e9b2dfe4690/b16f55a3-e312-45fa-a45f-1850db188063"
-					(reference "D53")
+					(reference "D1")
 					(unit 1)
 				)
@@
 		(dnp no)
 		(fields_autoplaced yes)
-		(property "Reference" "D42"
+		(property "Reference" "D36"
 			(at 281.94 185.0546 0)
 			(effects
@@
 			(project "Projet-ELEC-GISTRE"
 				(path "/88219bad-2ec7-47f4-a09d-0e9b2dfe4690/b16f55a3-e312-45fa-a45f-1850db188063"
-					(reference "D42")
+					(reference "D36")
 					(unit 1)
 				)
@@
 		(dnp no)
 		(fields_autoplaced yes)
-		(property "Reference" "D27"
+		(property "Reference" "D23"
 			(at 256.54 134.2546 0)
 			(effects
@@
 			(project "Projet-ELEC-GISTRE"
 				(path "/88219bad-2ec7-47f4-a09d-0e9b2dfe4690/b16f55a3-e312-45fa-a45f-1850db188063"
-					(reference "D27")
+					(reference "D23")
 					(unit 1)
 				)
@@
 		(dnp no)
 		(fields_autoplaced yes)
-		(property "Reference" "D36"
+		(property "Reference" "D42"
 			(at 129.54 185.0546 0)
 			(effects
@@
 			(project "Projet-ELEC-GISTRE"
 				(path "/88219bad-2ec7-47f4-a09d-0e9b2dfe4690/b16f55a3-e312-45fa-a45f-1850db188063"
-					(reference "D36")
+					(reference "D42")
 					(unit 1)
 				)
@@
 		(dnp no)
 		(fields_autoplaced yes)
-		(property "Reference" "D40"
+		(property "Reference" "D38"
 			(at 231.14 185.0546 0)
 			(effects
@@
 			(project "Projet-ELEC-GISTRE"
 				(path "/88219bad-2ec7-47f4-a09d-0e9b2dfe4690/b16f55a3-e312-45fa-a45f-1850db188063"
-					(reference "D40")
+					(reference "D38")
 					(unit 1)
 				)
@@
 		(dnp no)
 		(fields_autoplaced yes)
-		(property "Reference" "D24"
+		(property "Reference" "D26"
 			(at 180.34 134.2546 0)
 			(effects
@@
 			(project "Projet-ELEC-GISTRE"
 				(path "/88219bad-2ec7-47f4-a09d-0e9b2dfe4690/b16f55a3-e312-45fa-a45f-1850db188063"
-					(reference "D24")
-					(unit 1)
-				)
-			)
-		)
-	)
-	(symbol
-		(lib_id "Device:D")
-		(at 309.88 232.41 90)
-		(unit 1)
-		(exclude_from_sim no)
-		(in_bom yes)
-		(on_board yes)
-		(dnp no)
-		(fields_autoplaced yes)
-		(property "Reference" "D102"
-			(at 312.42 231.1399 90)
-			(effects
-				(font
-					(size 1.27 1.27)
-				)
-				(justify right)
-			)
-		)
-		(property "Value" "D"
-			(at 312.42 233.6799 90)
-			(effects
-				(font
-					(size 1.27 1.27)
-				)
-				(justify right)
-			)
-		)
-		(property "Footprint" ""
-			(at 309.88 232.41 0)
-			(effects
-				(font
-					(size 1.27 1.27)
-				)
-				(hide yes)
-			)
-		)
-		(property "Datasheet" "~"
-			(at 309.88 232.41 0)
-			(effects
-				(font
-					(size 1.27 1.27)
-				)
-				(hide yes)
-			)
-		)
-		(property "Description" "Diode"
-			(at 309.88 232.41 0)
-			(effects
-				(font
-					(size 1.27 1.27)
-				)
-				(hide yes)
-			)
-		)
-		(property "Sim.Device" "D"
-			(at 309.88 232.41 0)
-			(effects
-				(font
-					(size 1.27 1.27)
-				)
-				(hide yes)
-			)
-		)
-		(property "Sim.Pins" "1=K 2=A"
-			(at 309.88 232.41 0)
-			(effects
-				(font
-					(size 1.27 1.27)
-				)
-				(hide yes)
-			)
-		)
-		(pin "2"
-		)
-		(pin "1"
-		)
-		(instances
-			(project ""
-				(path "/88219bad-2ec7-47f4-a09d-0e9b2dfe4690/b16f55a3-e312-45fa-a45f-1850db188063"
-					(reference "D102")
+					(reference "D26")
 					(unit 1)
 				)
